File: nRF-devboard.kicad_sch (KiCad schematic)
At the start: 0 parts

Commit message: finished making nPM1300 symbol and wiring done :D
Parts:
- added C1, C2, C3, C5, C6: 10uF, Capacitor_SMD:C_0805_2012Metric_Pad1.18x1.45mm_HandSolder, symbol Device:C_Small
- added C4: 1uF, Capacitor_SMD:C_0402_1005Metric_Pad0.74x0.62mm_HandSolder, symbol Device:C_Small
- added C7: 2.2uF, Capacitor_SMD:C_0805_2012Metric_Pad1.18x1.45mm_HandSolder, symbol Device:C_Small
- added J1: GT-USB-7010ASV, easyeda2kicad:USB-C-SMD_G-SWITCH_GT-USB-7010ASV, symbol easyeda2kicad:GT-USB-7010ASV
- added L1, L2: 2.2uH, Inductor_SMD:L_1008_2520Metric_Pad1.43x2.20mm_HandSolder, symbol Device:L_Small
- added LED1: TC5050RGBF08-3CJH-AF53A, easyeda2kicad:LED-SMD_6P-L5.0-W5.0-TL_TC5050RGBF08, symbol easyeda2kicad:TC5050RGBF08-3CJH-AF53A
- added R1, R2: 390k, Resistor_SMD:R_0402_1005Metric_Pad0.72x0.64mm_HandSolder, symbol Device:R_Small
- added R3, R4: 10k, Resistor_SMD:R_0402_1005Metric_Pad0.72x0.64mm_HandSolder, symbol Device:R_Small
- added U1: nPM1300, Package_DFN_QFN:QFN-32-1EP_5x5mm_P0.5mm_EP3.6x3.6mm, symbol nPM:nPM1300
- added U2: nRF52840, Package_DFN_QFN:Nordic_AQFN-73-1EP_7x7mm_P0.5mm, symbol MCU_Nordic:nRF52840
Connections:
- new net: LED1.4 (-), U1.27 (LED2)
- new net: LED1.5 (-), U1.26 (LED1)
- new net: LED1.6 (-), U1.25 (LED0)
- new net: J1.A6 (DP1), J1.B6 (DP2), U2.AD6 (D+)
- new net: J1.A7 (DN1), J1.B7 (DN2), U2.AD4 (D-)
- new net: L1.2, U1.3 (SW1)
- new net: R2.2, U1.17 (VSET1)
- new net: L2.2, U1.5 (SW2)
- new net: R1.2, U1.16 (VSET2)
- new net +2.7V: C5.1, L1.1, U1.1 (VOUT1), U2.A22 (VDD), U2.AD14 (VDD), U2.AD23 (VDD), U2.B1 (VDD), U2.W1 (VDD), U2.Y2 (VDDH)
- new net +3.3V: C6.1, L2.1, U1.32 (VOUT2)
- new net CC1: J1.A5 (CC1), U1.23 (CC1)
- new net CC2: J1.B5 (CC2), U1.24 (CC2)
- new net GND: C1.2, C2.2, C3.2, C4.2, C5.2, C6.2, C7.2, J1.1 (SHELL), J1.2 (SHELL), J1.3 (SHELL), J1.4 (SHELL), J1.A1B12 (GND), J1.B1A12 (GND), R1.1, R2.1, U1.2 (PVSS1), U1.33 (AVSS), U1.6 (PVSS2), U2.B7 (VSS), U2.EP (VSS), U2.F23 (VSS_PA)
- new net GPIO0: U1.7 (GPIO0)
- new net GPIO1: U1.8 (GPIO1)
- new net GPIO2: U1.9 (GPIO2)
- new net GPIO3: U1.10 (GPIO3)
- new net GPIO4: U1.11 (GPIO4)
- new net SCL: R3.1, U1.14 (SCL)
- new net SDA: R4.1, U1.13 (SDA)
- new net VBAT: C7.1, U1.19 (VBAT)
- new net VBUS: J1.A4B9 (VBUS), J1.B4A9 (VBUS), U1.21 (VBUS)
- new net VDDIO: U1.12 (VDDIO)
- new net VSYS: C1.1, C2.1, C3.1, C4.1, LED1.1 (+), LED1.2 (+), LED1.3 (+), R3.2, R4.2, U1.20 (VSYS), U1.22 (VBUSOUT), U1.4 (PVDD)
Other:
- note added: "both of these voltages are configurable in software, so these are the defaults"
